Commit message: Change the inertia value for each parts

File: omorobot_r1_mini_description/urdf/gazebo.urdf.xacro (robot description, xacro)
@@ -1,3 +1,24 @@
 <?xml version="1.0"?>
 <robot xmlns:xacro="http://wiki.ros.org/xacro">
+    <gazebo reference="l_wheel_link">
+        <mu1>200</mu1>
+        <mu2>200</mu2>
+        <kp>10000000.0</kp>
+        <kd>1.0</kd>
+        <!-- <minDepth>0.001</minDepth> -->
+    </gazebo>
+    <gazebo reference="r_wheel_link">
+        <mu1>200</mu1>
+        <mu2>200</mu2>
+        <kp>10000000.0</kp>
+        <kd>1.0</kd>
+        <!-- <minDepth>0.001</minDepth> -->
+    </gazebo>
+    <gazebo reference="caster_wheel">
+        <mu1>1</mu1>
+        <mu2>1</mu2>
+        <kp>10000000.0</kp>
+        <kd>1.0</kd>
+        <!-- <minDepth>0.001</minDepth> -->
+    </gazebo>
 </robot>

File: omorobot_r1_mini_description/urdf/lidar_sensor.urdf.xacro (robot description, xacro)
@@ -11,13 +11,14 @@
                 </visual>
                 <collision>
-                    <origin xyz="0 0 0" rpy="0 0 0"/>
+                    <origin xyz="-0.015 0 0.035" rpy="0 0 0"/>
                     <geometry>
-                        <mesh filename="package://omorobot_r1_mini_description/meshes/ydlidar_assy.dae" scale="1 1 1"/>
+                        <!-- <mesh filename="package://omorobot_r1_mini_description/meshes/ydlidar_assy.dae" scale="1 1 1"/> -->
+                        <box size="0.1 0.07 0.04"/>
                     </geometry>
                 </collision>
                 <inertial>
-                    <origin xyz="0 0 0" rpy="0 0 0"/>
+                    <origin xyz="-0.015 0 0.035" rpy="0 0 0"/>
                     <mass value="0.5"/>
-                    <xacro:box_inertia m="0.5" x="0.154" y="0.130" z="0.04"/>
+                    <xacro:box_inertia m="0.5" x="0.1" y="0.07" z="0.04"/>
                 </inertial>
             </link>

File: omorobot_r1_mini_description/urdf/mobile_base.urdf.xacro (robot description, xacro)
@@ -10,13 +10,14 @@
             </visual>
             <collision>
-                <origin xyz="0 0 0" rpy="0 0 0"/>
+                <origin xyz="-0.0205 0 -0.003" rpy="0 0 0"/>
                 <geometry>
-                    <mesh filename="package://omorobot_r1_mini_description/meshes/body_assy.dae" scale="1 1 1"/>
+                    <!-- <mesh filename="package://omorobot_r1_mini_description/meshes/body_assy.dae" scale="1 1 1"/> -->
+                    <box size="0.108 0.13 0.038"/>
                 </geometry>
             </collision>
             <inertial>
-                <origin xyz="0 0 0" rpy="0 0 0"/>
-                <mass value="0.5"/>
-                <xacro:box_inertia m="0.5" x="0.154" y="0.130" z="0.04"/>
+                <origin xyz="-0.0205 0 -0.003" rpy="0 0 0"/>
+                <mass value="1.0"/>
+                <xacro:box_inertia m="0.5" x="0.108" y="0.13" z="0.038"/>
             </inertial>
         </link>
@@ -35,13 +36,14 @@
                 </visual>
                 <collision>
-                    <origin xyz="0 0 0" rpy="0 0 ${dir*pi/2}"/>
+                    <origin xyz="0 0 0" rpy="${pi/2} 0 0"/>
                     <geometry>
-                        <mesh filename="package://omorobot_r1_mini_description/meshes/wheel_assy.dae" scale="1 1 1"/>
+                        <!-- <mesh filename="package://omorobot_r1_mini_description/meshes/wheel_assy.dae" scale="1 1 1"/> -->
+                        <cylinder radius="${0.065/2}" length="0.027"/>
                     </geometry>
                 </collision>
                 <inertial>
                     <origin xyz="0 0 0" rpy="0 0 0"/>
-                    <mass value="0.1"/>
-                    <xacro:cylinder_inertia m="0.1" r="${0.065/2}" h="0.027"/>
+                    <mass value="0.01"/>
+                    <xacro:cylinder_inertia m="0.01" r="${0.065/2}" h="0.027"/>
                 </inertial>
             </link>
@@ -69,7 +71,7 @@
             </collision>
             <inertial>
-                <origin xyz="0 0 0" rpy="0 0 0"/>
-                <mass value="0.1"/>
-                <xacro:box_inertia m="0.1" x="0.154" y="0.130" z="0.04"/>
+                <origin xyz="-0.0205 0 0.019" rpy="0 0 0"/>
+                <mass value="0.2"/>
+                <xacro:box_inertia m="0.2" x="0.108" y="0.13" z="0.038"/>
             </inertial>
         </link>
@@ -88,13 +90,14 @@
                 </visual>
                 <collision>
-                    <origin xyz="0 0 0" rpy="0 0 0"/>
+                    <origin xyz="0 0 -0.0045" rpy="0 0 0"/>
                     <geometry>
-                        <mesh filename="package://omorobot_r1_mini_description/meshes/caster_wheel_mount.dae" scale="1 1 1"/>
+                        <!-- <mesh filename="package://omorobot_r1_mini_description/meshes/caster_wheel_mount.dae" scale="1 1 1"/> -->
+                        <box size="0.032 0.04 0.009"/>
                     </geometry>
                 </collision>
                 <inertial>
-                    <origin xyz="0 0 0" rpy="0 0 0"/>
+                    <origin xyz="0 0 -0.0045" rpy="0 0 0"/>
                     <mass value="0.1"/>
-                    <xacro:cylinder_inertia m="0.1" r="${0.065/2}" h="0.027"/>
+                    <xacro:box_inertia m="0.2" x="0.032" y="0.04" z="0.009"/>
                 </inertial>
             </link>
@@ -112,13 +115,14 @@
                 </visual>
                 <collision>
-                    <origin xyz="0 0 0" rpy="0 0 0"/>
+                    <origin xyz="0 0 -0.001" rpy="0 0 0"/>
                     <geometry>
-                        <mesh filename="package://omorobot_r1_mini_description/meshes/caster_wheel_rotate.dae" scale="1 1 1"/>
+                        <!-- <mesh filename="package://omorobot_r1_mini_description/meshes/caster_wheel_rotate.dae" scale="1 1 1"/> -->
+                        <cylinder radius="0.015" length="0.004"/>
                     </geometry>
                 </collision>
                 <inertial>
-                    <origin xyz="0 0 0" rpy="0 0 0"/>
+                    <origin xyz="0 0 -0.001" rpy="0 0 0"/>
                     <mass value="0.1"/>
-                    <xacro:cylinder_inertia m="0.1" r="${0.065/2}" h="0.027"/>
+                    <xacro:cylinder_inertia m="0.1" r="0.015" h="0.004"/>
                 </inertial>
             </link>
@@ -137,13 +141,14 @@
                 </visual>
                 <collision>
-                    <origin xyz="0 0 0" rpy="0 0 0"/>
+                    <origin xyz="0 0 0" rpy="${pi/2} 0 0"/>
                     <geometry>
-                        <mesh filename="package://omorobot_r1_mini_description/meshes/caster_wheel.dae" scale="1 1 1"/>
+                        <!-- <mesh filename="package://omorobot_r1_mini_description/meshes/caster_wheel.dae" scale="1 1 1"/> -->
+                        <cylinder radius="0.016" length="0.014"/>
                     </geometry>
                 </collision>
                 <inertial>
-                    <origin xyz="0 0 0" rpy="0 0 0"/>
+                    <origin xyz="0 0 0" rpy="${pi/2} 0 0"/>
                     <mass value="0.1"/>
-                    <xacro:cylinder_inertia m="0.1" r="${0.065/2}" h="0.027"/>
+                    <xacro:cylinder_inertia m="0.1" r="0.016" h="0.014"/>
                 </inertial>
             </link>

Commit message: Add diff_drive_controller and bringup_gazebo.launch

File: omorobot_r1_mini_description/urdf/gazebo.urdf.xacro (robot description, xacro)
@@ -22,3 +22,11 @@
         <!-- <minDepth>0.001</minDepth> -->
     </gazebo>
+    <gazebo>
+        <plugin name="gazebo_ros_control" filename="libgazebo_ros_control.so">
+            <robotNamespace></robotNamespace>
+            <robotSimType>gazebo_ros_control/DefaultRobotHWSim</robotSimType>
+            <controlPeriod>0.001</controlPeriod>
+            <legacyModeNS>false</legacyModeNS>
+        </plugin>
+    </gazebo>
 </robot>

File: omorobot_r1_mini_description/urdf/lidar_sensor.urdf.xacro (robot description, xacro)
@@ -19,6 +19,6 @@
                 <inertial>
                     <origin xyz="-0.015 0 0.035" rpy="0 0 0"/>
-                    <mass value="0.5"/>
-                    <xacro:box_inertia m="0.5" x="0.1" y="0.07" z="0.04"/>
+                    <mass value="0.05"/>
+                    <xacro:box_inertia m="0.05" x="0.1" y="0.07" z="0.04"/>
                 </inertial>
             </link>

File: omorobot_r1_mini_description/urdf/mobile_base.urdf.xacro (robot description, xacro)
@@ -54,4 +54,5 @@
                 <axis xyz="0 1 0"/>
             </joint>
+            <xacro:insert_velocity_transmission name="${prefix}_wheel_joint"/>
         </xacro:macro>
         <xacro:insert_wheel prefix="l" dir="1"/>

Commit message: Add lidar sensor in gazebo

File: omorobot_r1_mini_description/urdf/gazebo.urdf.xacro (robot description, xacro)
@@ -30,3 +30,34 @@
         </plugin>
     </gazebo>
+    <gazebo reference="lidar_link">
+        <sensor type="gpu_ray" name="lidar_sensor">
+            <pose>0 0 0 0 0 0</pose>
+            <visualize>true</visualize>
+            <update_rate>8</update_rate>
+            <ray>
+                <scan>
+                    <horizontal>
+                        <samples>576</samples>
+                        <resolution>1</resolution>
+                        <min_angle>${-180/180*pi}</min_angle>
+                        <max_angle>${180/180*pi}</max_angle>
+                    </horizontal>
+                </scan>
+                <range>
+                    <min>0.10</min>
+                    <max>12.0</max>
+                    <resolution>0.01</resolution>
+                </range>
+                <noise>
+                    <type>gaussian</type>
+                    <mean>0.0</mean>
+                    <stddev>0.01</stddev>
+                </noise>
+            </ray>
+            <plugin name="gazebo_ros_head_hokuyo_controller" filename="libgazebo_ros_gpu_laser.so">
+                <topicName>scan</topicName>
+                <frameName>lidar_link</frameName>
+            </plugin>
+        </sensor>
+    </gazebo>
 </robot>

File: omorobot_r1_mini_description/urdf/lidar_sensor.urdf.xacro (robot description, xacro)
@@ -19,5 +19,5 @@
                 <inertial>
                     <origin xyz="-0.015 0 0.035" rpy="0 0 0"/>
-                    <mass value="0.05"/>
+                    <mass value="0.2"/>
                     <xacro:box_inertia m="0.05" x="0.1" y="0.07" z="0.04"/>
                 </inertial>

File: omorobot_r1_mini_description/urdf/mobile_base.urdf.xacro (robot description, xacro)
@@ -99,6 +99,6 @@
                 <inertial>
                     <origin xyz="0 0 -0.0045" rpy="0 0 0"/>
-                    <mass value="0.1"/>
-                    <xacro:box_inertia m="0.2" x="0.032" y="0.04" z="0.009"/>
+                    <mass value="0.02"/>
+                    <xacro:box_inertia m="0.02" x="0.032" y="0.04" z="0.009"/>
                 </inertial>
             </link>
@@ -124,6 +124,6 @@
                 <inertial>
                     <origin xyz="0 0 -0.001" rpy="0 0 0"/>
-                    <mass value="0.1"/>
-                    <xacro:cylinder_inertia m="0.1" r="0.015" h="0.004"/>
+                    <mass value="0.02"/>
+                    <xacro:cylinder_inertia m="0.02" r="0.015" h="0.004"/>
                 </inertial>
             </link>
@@ -150,6 +150,6 @@
                 <inertial>
                     <origin xyz="0 0 0" rpy="${pi/2} 0 0"/>
-                    <mass value="0.1"/>
-                    <xacro:cylinder_inertia m="0.1" r="0.016" h="0.014"/>
+                    <mass value="0.02"/>
+                    <xacro:cylinder_inertia m="0.02" r="0.016" h="0.014"/>
                 </inertial>
             </link>

Commit message: Add IMU in Gazebo

File: omorobot_r1_mini_description/urdf/gazebo.urdf.xacro (robot description, xacro)
@@ -61,3 +61,23 @@
         </sensor>
     </gazebo>
+    <gazebo reference="imu_link">
+        <gravity>true</gravity>
+        <sensor name="imu_sensor" type="imu">
+            <always_on>true</always_on>
+            <update_rate>100</update_rate>
+            <visualize>true</visualize>
+            <topic>__default_topic__</topic>
+            <plugin filename="libgazebo_ros_imu_sensor.so" name="imu_plugin">
+                <topicName>imu</topicName>
+                <bodyName>imu_link</bodyName>
+                <updateRateHZ>25.0</updateRateHZ>
+                <gaussianNoise>0.01</gaussianNoise>
+                <xyzOffset>0 0 0</xyzOffset>
+                <rpyOffset>0 0 0</rpyOffset>
+                <frameName>imu_link</frameName>
+                <initialOrientationAsReference>false</initialOrientationAsReference>
+            </plugin>
+            <pose>0 0 0 0 0 0</pose>
+        </sensor>
+    </gazebo>
 </robot>

File: omorobot_r1_mini_description/urdf/mobile_base.urdf.xacro (robot description, xacro)
@@ -43,5 +43,5 @@
                 </collision>
                 <inertial>
-                    <origin xyz="0 0 0" rpy="0 0 0"/>
+                    <origin xyz="0 0 0" rpy="${pi/2} 0 0"/>
                     <mass value="0.01"/>
                     <xacro:cylinder_inertia m="0.01" r="${0.065/2}" h="0.027"/>
@@ -164,4 +164,10 @@
             <origin xyz="-0.10375 0 0.01425" rpy="0 0 0"/>
         </xacro:insert_caster_wheel>
+        <link name="imu_link"/>
+        <joint name="imu_link_fixed" type="fixed">
+            <parent link="base_link"/>
+            <child link="imu_link"/>
+            <origin xyz="0 0 0" rpy="0 0 0"/>
+        </joint>
     </xacro:macro>
 </robot>
